File: KiCad/C3/Unified-Daughterboard.kicad_sch (KiCad schematic)
At the start: 30 parts, among them J1 TYPE-C-31-M12_13, J3 Battery, J4 Conn_01x06, Q1 2N7002, SW1 PWR, U1 TPD4E05U06DQAR, U2 BQ24075

Commit message: STEP export
Parts:
- J4: footprint Connector_JST:JST_SH_SM06B-SRSS-TB_1x06-1MP_P1.00mm_Horizontal -> PCM_marbastlib-various:Molex_Pico-EZmate_78171-5006_1x06-1MP_P1.20mm_Vertical
Changed lines of the file:
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@@
 			)
 		)
-		(property "Footprint" "Connector_JST:JST_SH_SM06B-SRSS-TB_1x06-1MP_P1.00mm_Horizontal"
+		(property "Footprint" "PCM_marbastlib-various:Molex_Pico-EZmate_78171-5006_1x06-1MP_P1.20mm_Vertical"
 			(at 241.3 80.01 0)
 			(effects
